File: Heizung.sch (EAGLE design)
At the start: 40 parts, among them IC1 MEGA8-PTQFP, Q2 2N7002, Q3 2N7002

Commit message: additional ground on power side, outline fixed
Parts:
- added _GND: WAGO_243, common:WAGO_243
- renumbered BGND to B_GND
Connections:
- net GND: now also _GND.1
Changed lines of the file:
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@@
 <setting verticaltext="up"/>
 </settings>
-<grid distance="0.1" unitdist="inch" unit="inch" style="lines" multiple="1" display="no" altdistance="0.05" altunitdist="inch" altunit="inch"/>
+<grid distance="0.1" unitdist="inch" unit="inch" style="lines" multiple="1" display="no" altdistance="0.01" altunitdist="inch" altunit="inch"/>
 <layers>
 <layer number="1" name="Top" color="4" fill="1" visible="no" active="no"/>
@@
 </class>
 <class number="1" name="wires" width="0.5" drill="0">
+<clearance class="1" value="0.35"/>
 </class>
 </classes>
@@
 <part name="C3" library="common" deviceset="C" device="C0603" value="15n"/>
 <part name="C1" library="common" deviceset="CP" device="1206" value="0.1µ"/>
-<part name="BGND" library="common" deviceset="WAGO_243" device="" value="WAGO_243"/>
+<part name="B_GND" library="common" deviceset="WAGO_243" device="" value="WAGO_243"/>
 <part name="B_24V" library="common" deviceset="WAGO_243" device="" value="WAGO_243"/>
 <part name="H1V" library="common" deviceset="PINHD-1X1" device="" value="WAGO_243"/>
@@
 <part name="R5" library="common" deviceset="R-EU_" device="M0805"/>
 <part name="R6" library="common" deviceset="R-EU_" device="M0805"/>
+<part name="_GND" library="common" deviceset="WAGO_243" device="" value="WAGO_243"/>
 </parts>
 <sheets>
@@
 <instance part="C3" gate="G$1" x="25.4" y="63.5" rot="R90"/>
 <instance part="C1" gate="G$1" x="33.02" y="83.82"/>
-<instance part="BGND" gate="G$1" x="15.24" y="99.06" smashed="yes">
+<instance part="B_GND" gate="G$1" x="15.24" y="99.06" smashed="yes">
 <attribute name="NAME" x="8.89" y="102.235" size="1.778" layer="95"/>
 </instance>
@@
 <instance part="R5" gate="G$1" x="132.08" y="93.98"/>
 <instance part="R6" gate="G$1" x="132.08" y="99.06"/>
+<instance part="_GND" gate="G$1" x="22.86" y="99.06" smashed="yes">
+<attribute name="NAME" x="16.51" y="102.235" size="1.778" layer="95"/>
+</instance>
 </instances>
 <busses>
@@
 <pinref part="C1" gate="G$1" pin="-"/>
 <wire x1="33.02" y1="78.74" x2="43.18" y2="78.74" width="0.1524" layer="91"/>
-<pinref part="BGND" gate="G$1" pin="1"/>
+<pinref part="B_GND" gate="G$1" pin="1"/>
 <wire x1="12.7" y1="99.06" x2="12.7" y2="93.98" width="0.1524" layer="91"/>
 <wire x1="12.7" y1="93.98" x2="12.7" y2="48.26" width="0.1524" layer="91"/>
@@
 <wire x1="27.94" y1="96.52" x2="27.94" y2="93.98" width="0.1524" layer="91"/>
 <junction x="27.94" y="93.98"/>
-</segment>
-</net>
+<pinref part="_GND" gate="G$1" pin="1"/>
+<wire x1="20.32" y1="99.06" x2="12.7" y2="99.06" width="0.1524" layer="91"/>
+<junction x="12.7" y="99.06"/>
+</segment>
+</net>

Commit message: Update auf 2.4
2-Draht-Klemmen verwendet und gedreht
Wagoklemmen nach innen gedreht
Parts:
- removed H1, H1V, H2, H2V: WAGO_243, common:PINHD-1X1
- added JP1, JP2: (no value), common:PINHD-1X2LEVER
- renumbered DT1 to 1W_1, DT1G to GND1, DT2 to 1W_2, DT2G to GND2
Connections:
- net N$1: now also JP1.1, JP2.1; no longer H1V.1, H2V.1
- net N$19: now also JP1.2; no longer H1.1
- net N$33: now also JP2.2; no longer H2.1
Changed lines of the file:
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@@
 <clearance class="1" value="0.35"/>
+</class>
+<class number="2" name="p24" width="1" drill="0">
+<clearance class="2" value="0.4"/>
 </class>
 </classes>
@@
 <part name="B_GND" library="common" deviceset="WAGO_243" device="" value="WAGO_243"/>
 <part name="B_24V" library="common" deviceset="WAGO_243" device="" value="WAGO_243"/>
-<part name="H1V" library="common" deviceset="PINHD-1X1" device="" value="WAGO_243"/>
-<part name="H1" library="common" deviceset="PINHD-1X1" device="" value="WAGO_243"/>
 <part name="Q2" library="common" deviceset="2N7002" device=""/>
 <part name="B_5V" library="common" deviceset="WAGO_243" device="" value="WAGO_243"/>
-<part name="DT1" library="common" deviceset="WAGO_243" device="" value="WAGO_243"/>
-<part name="DT1G" library="common" deviceset="WAGO_243" device="" value="WAGO_243"/>
-<part name="DT2" library="common" deviceset="WAGO_243" device="" value="WAGO_243"/>
-<part name="DT2G" library="common" deviceset="WAGO_243" device="" value="WAGO_243"/>
+<part name="1W_1" library="common" deviceset="WAGO_243" device="" value="WAGO_243"/>
+<part name="GND1" library="common" deviceset="WAGO_243" device="" value="WAGO_243"/>
+<part name="1W_2" library="common" deviceset="WAGO_243" device="" value="WAGO_243"/>
+<part name="GND2" library="common" deviceset="WAGO_243" device="" value="WAGO_243"/>
 <part name="I_5V" library="common" deviceset="WAGO_243" device="" value="WAGO_243"/>
 <part name="I_GND" library="common" deviceset="WAGO_243" device="" value="WAGO_243"/>
@@
 <part name="D3" library="common" deviceset="ESD_DIODES" device=""/>
 <part name="Q3" library="common" deviceset="2N7002" device=""/>
-<part name="H2V" library="common" deviceset="PINHD-1X1" device="" value="WAGO_243"/>
-<part name="H2" library="common" deviceset="PINHD-1X1" device="" value="WAGO_243"/>
 <part name="R5" library="common" deviceset="R-EU_" device="M0805"/>
 <part name="R6" library="common" deviceset="R-EU_" device="M0805"/>
 <part name="_GND" library="common" deviceset="WAGO_243" device="" value="WAGO_243"/>
+<part name="JP1" library="common" deviceset="PINHD-1X2" device="LEVER"/>
+<part name="JP2" library="common" deviceset="PINHD-1X2" device="LEVER"/>
 </parts>
 <sheets>
@@
 <attribute name="NAME" x="8.89" y="125.095" size="1.778" layer="95"/>
 </instance>
-<instance part="H1V" gate="G$1" x="53.34" y="121.92" smashed="yes">
-<attribute name="NAME" x="46.99" y="125.095" size="1.778" layer="95"/>
-</instance>
-<instance part="H1" gate="G$1" x="53.34" y="111.76" smashed="yes">
-<attribute name="NAME" x="46.99" y="114.935" size="1.778" layer="95"/>
-</instance>
 <instance part="Q2" gate="&gt;NAME" x="53.34" y="99.06" rot="MR0"/>
 <instance part="B_5V" gate="G$1" x="15.24" y="111.76"/>
-<instance part="DT1" gate="G$1" x="144.78" y="66.04"/>
-<instance part="DT1G" gate="G$1" x="144.78" y="55.88"/>
-<instance part="DT2" gate="G$1" x="144.78" y="43.18"/>
-<instance part="DT2G" gate="G$1" x="144.78" y="33.02"/>
+<instance part="1W_1" gate="G$1" x="144.78" y="66.04"/>
+<instance part="GND1" gate="G$1" x="144.78" y="55.88"/>
+<instance part="1W_2" gate="G$1" x="144.78" y="43.18"/>
+<instance part="GND2" gate="G$1" x="144.78" y="33.02"/>
 <instance part="I_5V" gate="G$1" x="134.62" y="116.84" smashed="yes">
 <attribute name="NAME" x="128.27" y="120.015" size="1.778" layer="95"/>
@@
 <instance part="D3" gate="G$1" x="149.86" y="104.14"/>
 <instance part="Q3" gate="&gt;NAME" x="35.56" y="99.06" rot="MR0"/>
-<instance part="H2V" gate="G$1" x="35.56" y="121.92" smashed="yes">
-<attribute name="NAME" x="29.21" y="125.095" size="1.778" layer="95"/>
-</instance>
-<instance part="H2" gate="G$1" x="35.56" y="111.76" smashed="yes">
-<attribute name="NAME" x="29.21" y="114.935" size="1.778" layer="95"/>
-</instance>
 <instance part="R5" gate="G$1" x="132.08" y="93.98"/>
 <instance part="R6" gate="G$1" x="132.08" y="99.06"/>
@@
 <attribute name="NAME" x="16.51" y="102.235" size="1.778" layer="95"/>
 </instance>
+<instance part="JP1" gate="G$1" x="53.34" y="119.38"/>
+<instance part="JP2" gate="G$1" x="35.56" y="119.38"/>
 </instances>
 <busses>
@@
 <pinref part="I_GND" gate="G$1" pin="1"/>
 <wire x1="142.24" y1="78.74" x2="142.24" y2="88.9" width="0.1524" layer="91"/>
-<pinref part="DT1G" gate="G$1" pin="1"/>
+<pinref part="GND1" gate="G$1" pin="1"/>
 <wire x1="142.24" y1="88.9" x2="142.24" y2="106.68" width="0.1524" layer="91"/>
 <wire x1="142.24" y1="106.68" x2="142.24" y2="121.92" width="0.1524" layer="91"/>
 <wire x1="137.16" y1="55.88" x2="142.24" y2="55.88" width="0.1524" layer="91"/>
-<pinref part="DT2G" gate="G$1" pin="1"/>
+<pinref part="GND2" gate="G$1" pin="1"/>
 <wire x1="142.24" y1="33.02" x2="137.16" y2="33.02" width="0.1524" layer="91"/>
 <wire x1="137.16" y1="33.02" x2="137.16" y2="55.88" width="0.1524" layer="91"/>
@@
 </segment>
 </net>
-<net name="N$1" class="1">
-<segment>
-<pinref part="H1V" gate="G$1" pin="1"/>
+<net name="N$1" class="2">
+<segment>
 <wire x1="12.7" y1="121.92" x2="33.02" y2="121.92" width="0.1524" layer="91"/>
 <pinref part="B_24V" gate="G$1" pin="1"/>
-<pinref part="H2V" gate="G$1" pin="1"/>
+<pinref part="JP1" gate="G$1" pin="1"/>
+<pinref part="JP2" gate="G$1" pin="1"/>
 <wire x1="33.02" y1="121.92" x2="50.8" y2="121.92" width="0.1524" layer="91"/>
 <junction x="33.02" y="121.92"/>
 </segment>
 </net>
-<net name="N$19" class="0">
-<segment>
-<pinref part="H1" gate="G$1" pin="1"/>
+<net name="N$19" class="2">
+<segment>
 <pinref part="Q2" gate="&gt;NAME" pin="D"/>
-<wire x1="50.8" y1="111.76" x2="45.72" y2="111.76" width="0.1524" layer="91"/>
-<wire x1="45.72" y1="111.76" x2="45.72" y2="101.6" width="0.1524" layer="91"/>
+<wire x1="45.72" y1="119.38" x2="45.72" y2="101.6" width="0.1524" layer="91"/>
+<pinref part="JP1" gate="G$1" pin="2"/>
+<wire x1="45.72" y1="119.38" x2="50.8" y2="119.38" width="0.1524" layer="91"/>
 </segment>
 </net>
@@
 <segment>
 <pinref part="D1" gate="G$1" pin="K1"/>
-<pinref part="DT1" gate="G$1" pin="1"/>
+<pinref part="1W_1" gate="G$1" pin="1"/>
 <wire x1="132.08" y1="53.34" x2="132.08" y2="66.04" width="0.1524" layer="91"/>
 <wire x1="132.08" y1="66.04" x2="142.24" y2="66.04" width="0.1524" layer="91"/>
@@
 <segment>
 <pinref part="D1" gate="G$1" pin="K2"/>
-<pinref part="DT2" gate="G$1" pin="1"/>
+<pinref part="1W_2" gate="G$1" pin="1"/>
 <wire x1="132.08" y1="43.18" x2="142.24" y2="43.18" width="0.1524" layer="91"/>
 <pinref part="IC1" gate="G$1" pin="PD3(INT1)"/>
@@
 </segment>
 </net>
-<net name="N$33" class="0">
-<segment>
-<pinref part="H2" gate="G$1" pin="1"/>
-<wire x1="33.02" y1="111.76" x2="25.4" y2="111.76" width="0.1524" layer="91"/>
+<net name="N$33" class="2">
+<segment>
+<wire x1="33.02" y1="119.38" x2="27.94" y2="119.38" width="0.1524" layer="91"/>
 <pinref part="Q3" gate="&gt;NAME" pin="D"/>
-<wire x1="25.4" y1="111.76" x2="25.4" y2="101.6" width="0.1524" layer="91"/>
-<wire x1="25.4" y1="101.6" x2="27.94" y2="101.6" width="0.1524" layer="91"/>
-</segment>
-</net>
+<wire x1="27.94" y1="119.38" x2="27.94" y2="101.6" width="0.1524" layer="91"/>
+<pinref part="JP2" gate="G$1" pin="2"/>
+</segment>
+</net>

Commit message: Längere Pads für CPU
Parts:
- removed P1, P1G, P2, P2G, P3, P3G, P4, P4G: (no value), common:PINHD-1X1
- added JP3, JP4, JP5, JP6: (no value), common:PINHD-1X2LEVER
Connections:
- net B1: now also JP3.2; no longer P1.1
- net B2: now also JP4.2; no longer P2.1
- net B3: now also JP5.2; no longer P3.1
- net B4: now also JP6.2; no longer P4.1
- net GND: now also JP3.1, JP4.1, JP5.1, JP6.1; no longer P1G.1, P2G.1, P3G.1, P4G.1
Changed lines of the file:
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@@
 <part name="R3" library="common" deviceset="R-EU_" device="M0805"/>
 <part name="R4" library="common" deviceset="R-EU_" device="M0805"/>
-<part name="P1" library="common" deviceset="PINHD-1X1" device=""/>
-<part name="P2" library="common" deviceset="PINHD-1X1" device=""/>
-<part name="P3" library="common" deviceset="PINHD-1X1" device=""/>
-<part name="P4" library="common" deviceset="PINHD-1X1" device=""/>
-<part name="P1G" library="common" deviceset="PINHD-1X1" device=""/>
-<part name="P2G" library="common" deviceset="PINHD-1X1" device=""/>
-<part name="P3G" library="common" deviceset="PINHD-1X1" device=""/>
-<part name="P4G" library="common" deviceset="PINHD-1X1" device=""/>
 <part name="D2" library="common" deviceset="ESD_DIODES" device=""/>
 <part name="D3" library="common" deviceset="ESD_DIODES" device=""/>
@@
 <part name="JP1" library="common" deviceset="PINHD-1X2" device="LEVER"/>
 <part name="JP2" library="common" deviceset="PINHD-1X2" device="LEVER"/>
+<part name="JP3" library="common" deviceset="PINHD-1X2" device="LEVER"/>
+<part name="JP4" library="common" deviceset="PINHD-1X2" device="LEVER"/>
+<part name="JP5" library="common" deviceset="PINHD-1X2" device="LEVER"/>
+<part name="JP6" library="common" deviceset="PINHD-1X2" device="LEVER"/>
 </parts>
 <sheets>
@@
 <instance part="R3" gate="G$1" x="162.56" y="76.2" rot="R90"/>
 <instance part="R4" gate="G$1" x="162.56" y="91.44" rot="R90"/>
-<instance part="P1" gate="G$1" x="170.18" y="121.92" rot="R90"/>
-<instance part="P2" gate="G$1" x="170.18" y="106.68" rot="R90"/>
-<instance part="P3" gate="G$1" x="170.18" y="91.44" rot="R90"/>
-<instance part="P4" gate="G$1" x="170.18" y="76.2" rot="R90"/>
-<instance part="P1G" gate="G$1" x="162.56" y="58.42" rot="R90"/>
-<instance part="P2G" gate="G$1" x="172.72" y="58.42" rot="R90"/>
-<instance part="P3G" gate="G$1" x="172.72" y="45.72" rot="R90"/>
-<instance part="P4G" gate="G$1" x="162.56" y="45.72" rot="R90"/>
 <instance part="D2" gate="G$1" x="149.86" y="91.44" rot="R180"/>
 <instance part="D3" gate="G$1" x="149.86" y="104.14"/>
@@
 <instance part="JP1" gate="G$1" x="53.34" y="119.38"/>
 <instance part="JP2" gate="G$1" x="35.56" y="119.38"/>
+<instance part="JP3" gate="G$1" x="172.72" y="119.38"/>
+<instance part="JP4" gate="G$1" x="172.72" y="104.14"/>
+<instance part="JP5" gate="G$1" x="172.72" y="88.9"/>
+<instance part="JP6" gate="G$1" x="172.72" y="73.66"/>
 </instances>
 <busses>
@@
 <junction x="63.5" y="78.74"/>
 <pinref part="I_GND" gate="G$1" pin="1"/>
-<wire x1="142.24" y1="78.74" x2="142.24" y2="88.9" width="0.1524" layer="91"/>
+<wire x1="142.24" y1="81.28" x2="142.24" y2="88.9" width="0.1524" layer="91"/>
 <pinref part="GND1" gate="G$1" pin="1"/>
 <wire x1="142.24" y1="88.9" x2="142.24" y2="106.68" width="0.1524" layer="91"/>
@@
 <wire x1="134.62" y1="48.26" x2="134.62" y2="33.02" width="0.1524" layer="91"/>
 <junction x="134.62" y="33.02"/>
-<wire x1="142.24" y1="78.74" x2="154.94" y2="78.74" width="0.1524" layer="91"/>
-<wire x1="154.94" y1="78.74" x2="154.94" y2="50.8" width="0.1524" layer="91"/>
-<junction x="142.24" y="78.74"/>
-<pinref part="P4G" gate="G$1" pin="1"/>
-<wire x1="154.94" y1="50.8" x2="154.94" y2="38.1" width="0.1524" layer="91"/>
-<wire x1="154.94" y1="38.1" x2="162.56" y2="38.1" width="0.1524" layer="91"/>
-<wire x1="162.56" y1="38.1" x2="162.56" y2="43.18" width="0.1524" layer="91"/>
-<pinref part="P3G" gate="G$1" pin="1"/>
-<wire x1="162.56" y1="38.1" x2="172.72" y2="38.1" width="0.1524" layer="91"/>
-<wire x1="172.72" y1="38.1" x2="172.72" y2="43.18" width="0.1524" layer="91"/>
-<junction x="162.56" y="38.1"/>
-<pinref part="P1G" gate="G$1" pin="1"/>
-<wire x1="154.94" y1="50.8" x2="162.56" y2="50.8" width="0.1524" layer="91"/>
-<wire x1="162.56" y1="50.8" x2="162.56" y2="55.88" width="0.1524" layer="91"/>
-<junction x="154.94" y="50.8"/>
-<pinref part="P2G" gate="G$1" pin="1"/>
-<wire x1="162.56" y1="50.8" x2="172.72" y2="50.8" width="0.1524" layer="91"/>
-<wire x1="172.72" y1="50.8" x2="172.72" y2="55.88" width="0.1524" layer="91"/>
-<junction x="162.56" y="50.8"/>
 <pinref part="D2" gate="G$1" pin="AA"/>
 <wire x1="149.86" y1="88.9" x2="142.24" y2="88.9" width="0.1524" layer="91"/>
@@
 <wire x1="20.32" y1="99.06" x2="12.7" y2="99.06" width="0.1524" layer="91"/>
 <junction x="12.7" y="99.06"/>
+<wire x1="142.24" y1="78.74" x2="142.24" y2="81.28" width="0.1524" layer="91"/>
+<wire x1="142.24" y1="81.28" x2="165.1" y2="81.28" width="0.1524" layer="91"/>
+<pinref part="JP6" gate="G$1" pin="1"/>
+<wire x1="165.1" y1="81.28" x2="165.1" y2="76.2" width="0.1524" layer="91"/>
+<wire x1="165.1" y1="76.2" x2="170.18" y2="76.2" width="0.1524" layer="91"/>
+<pinref part="JP5" gate="G$1" pin="1"/>
+<wire x1="165.1" y1="81.28" x2="165.1" y2="91.44" width="0.1524" layer="91"/>
+<wire x1="165.1" y1="91.44" x2="170.18" y2="91.44" width="0.1524" layer="91"/>
+<junction x="165.1" y="81.28"/>
+<pinref part="JP4" gate="G$1" pin="1"/>
+<wire x1="165.1" y1="91.44" x2="165.1" y2="106.68" width="0.1524" layer="91"/>
+<wire x1="165.1" y1="106.68" x2="170.18" y2="106.68" width="0.1524" layer="91"/>
+<junction x="165.1" y="91.44"/>
+<pinref part="JP3" gate="G$1" pin="1"/>
+<wire x1="165.1" y1="106.68" x2="165.1" y2="121.92" width="0.1524" layer="91"/>
+<wire x1="165.1" y1="121.92" x2="170.18" y2="121.92" width="0.1524" layer="91"/>
+<junction x="165.1" y="106.68"/>
 </segment>
 </net>
@@
 <segment>
 <pinref part="R2" gate="G$1" pin="1"/>
-<pinref part="P1" gate="G$1" pin="1"/>
 <wire x1="162.56" y1="116.84" x2="170.18" y2="116.84" width="0.1524" layer="91"/>
 <wire x1="170.18" y1="116.84" x2="170.18" y2="119.38" width="0.1524" layer="91"/>
 <wire x1="170.18" y1="116.84" x2="175.26" y2="116.84" width="0.1524" layer="91"/>
 <junction x="170.18" y="116.84"/>
+<pinref part="JP3" gate="G$1" pin="2"/>
 </segment>
 <segment>
@@
 <segment>
 <pinref part="R1" gate="G$1" pin="1"/>
-<pinref part="P2" gate="G$1" pin="1"/>
 <wire x1="162.56" y1="101.6" x2="170.18" y2="101.6" width="0.1524" layer="91"/>
 <wire x1="170.18" y1="101.6" x2="170.18" y2="104.14" width="0.1524" layer="91"/>
 <wire x1="170.18" y1="101.6" x2="175.26" y2="101.6" width="0.1524" layer="91"/>
 <junction x="170.18" y="101.6"/>
+<pinref part="JP4" gate="G$1" pin="2"/>
 </segment>
 <segment>
@@
 <segment>
 <pinref part="R4" gate="G$1" pin="1"/>
-<pinref part="P3" gate="G$1" pin="1"/>
 <wire x1="162.56" y1="86.36" x2="170.18" y2="86.36" width="0.1524" layer="91"/>
 <wire x1="170.18" y1="86.36" x2="170.18" y2="88.9" width="0.1524" layer="91"/>
 <wire x1="170.18" y1="86.36" x2="175.26" y2="86.36" width="0.1524" layer="91"/>
 <junction x="170.18" y="86.36"/>
+<pinref part="JP5" gate="G$1" pin="2"/>
 </segment>
 <segment>
@@
 <segment>
 <pinref part="R3" gate="G$1" pin="1"/>
-<pinref part="P4" gate="G$1" pin="1"/>
 <wire x1="162.56" y1="71.12" x2="170.18" y2="71.12" width="0.1524" layer="91"/>
 <wire x1="170.18" y1="71.12" x2="170.18" y2="73.66" width="0.1524" layer="91"/>
 <wire x1="170.18" y1="71.12" x2="175.26" y2="71.12" width="0.1524" layer="91"/>
 <junction x="170.18" y="71.12"/>
-</segment>
-<segment>
+<pinref part="JP6" gate="G$1" pin="2"/>
+</segment>
+<segment>

Commit message: V2.7: add diode (for switching relays)
general clean-up
Parts:
- removed R1, R2, R3, R4: (no value), common:R-EU_M0805
- added D4: BAS40-05, common:BAS40-05
- renumbered B_24V to 24V, B_5V to 5V, I_5V to 5V_, I_CLK to CLK, I_DATA to DATA, I_GND to GND_, JP3 to J_1, JP4 to J_2, JP5 to J_3, JP6 to J_4
Connections:
- net 5V: no longer R1.2, R2.2, R3.2, R4.2
- net B1: now also D2.K2; no longer D3.K1, R2.1
- net B2: now also D2.K1; no longer D3.K2, R1.1
- net B3: now also D3.K1; no longer D2.K1, R4.1
- net B4: now also D3.K2; no longer D2.K2, R3.1
- net N$1: now also D4.C
- net N$19: now also D4.A2
- net N$33: now also D4.A1
